Commit message: second

File: urdf/mobile_robot.urdf (robot description, URDF)
Before this commit: robot mobilerobot, 1 links, 0 joints
Links:
- added link caster_support; collision box size=0.02 0.02 0.04; visual box size=0.02 0.02 0.04
- added link caster_wheel; collision cylinder length=0.005 radius=0.02; visual cylinder length=0.005 radius=0.02
- added link laser; collision box size=0.05 0.05 0.05; visual box size=0.05 0.05 0.05
- added link left_wheel; collision cylinder length=0.008 radius=0.024; visual cylinder length=0.008 radius=0.024
- added link right_wheel; collision cylinder length=0.008 radius=0.024; visual cylinder length=0.008 radius=0.024
- link base_link: geometry collision box size=0.13 0.1 0.078; visual box size=0.005 0.065 0.02
Joints:
- added joint caster_support_joint: type continuous, parent base_link, child caster_support, origin xyz=-0.065 0 -0.01 rpy=0 0 0, axis 0 0 1
- added joint caster_wheel_joint: type continuous, parent caster_support, child caster_wheel, origin xyz=-0.02 0 -0.02 rpy=-1.5708 0 0, axis 0 0 1
- added joint laser_joint: type fixed, parent base_link, child laser, origin xyz=0 0 0.051 rpy=0 0 0
- added joint left_wheel_joint: type continuous, parent base_link, child left_wheel, origin xyz=0 -0.054 -0.021 rpy=-1.5708 0 0, axis 0 0 1
- added joint right_wheel_joint: type continuous, parent base_link, child right_wheel, origin xyz=0 0.054 -0.021 rpy=-1.5708 0 0, axis 0 0 1
